File: test_stand_smd.sch (KiCad schematic (older format))
At the start: 22 parts, among them J1 Conn_01x05_Male, J2 USB_C_Receptacle_USB2.0, U1 ATSAMD21E, U2 AP2112K-3.3

Commit message: Added schematic comments
Parts:
- J1: value Conn_01x05_Male -> MA3 Abs. Rotary Enc. Connector
- SW_0: renamed from SW_HOME1; value SW_Push -> ZERO_SW
- U1: symbol trinket_m0:ATSAMD21E -> test_stand_smd-rescue:ATSAMD21E-trinket_m0
Connections:
- net HOME_SW renamed ZERO_SW
Other:
- note added: "(3.3k) / (1.7k + 3.3k) = 0.66"
- note added: "5.1k pulldown resistors used to\nindicate port is an upstream port\n(USB Type-C spec, allows for C to C cable usage)"
- note added: "Borrowed from Adafruit's \nTrinket M0 schematic"
- note added: "Power Indicator"
- note added: "Programmable LED"
- note added: "Same uC that the Adafruit\nTrinket M0 & QT PY use, \nwill likely get changed\ndue to chip shortage"
- note added: "Used in firmware to \n"zero" the position of \nthe MA3 encoder"
- note added: "Voltage divider to scale 5V\nanalog output of MA3 to\n3.3V analog input for \nuC"
- moved on the sheet: F1, J1, J2, R1, R2, R3, R4, R5, R6, R7, SW_0
